Commit message: gazebo package added

File: lab1_tut/src/urdf/one_shape.urdf (robot description, URDF)
Before this commit: robot myfirst, 2 links, 1 joints
Joints:
- joint rev1: axis 0.0 1.0 0.0 -> (none); limit lower=0.0 upper=30.0 effort=30.0 velocity=2.0 -> (none); type revolute -> fixed

File: macro_tutorial/src/model/combined_model.urdf.xacro (robot description, xacro)
@@ -4,12 +4,15 @@
      For more information, please see http://wiki.ros.org/sw_urdf_exporter -->
 <robot xmlns:xacro="http://ros.org/wiki/xacro" name="full_model">
-    <xacro:include filename="$(find macro_tutorial)/src/model/model.urdf.xacro"/>
-    <xacro:include filename="$(find gripper_pkg)/urdf/grip.urdf.xacro"/>
-    <xacro:rotating_base/>
-    <xacro:gripper/>
-    <joint name="attachment" type="fixed">
-        <origin xyz="0.0 0.1 0.125" rpy="0.0 0.0 0.0"/>
-        <parent link="inter_1"/>
-        <child link="grip_body"/>
-    </joint>
+    <xacro:macro name="combined_model">
+        <xacro:include filename="$(find macro_tutorial)/src/model/model.urdf.xacro"/>
+        <xacro:include filename="$(find gripper_pkg)/urdf/grip.urdf.xacro"/>
+        <xacro:rotating_base/>
+        <xacro:gripper/>
+        <joint name="attachment" type="fixed">
+            <origin xyz="0.0 0.1 0.125" rpy="0.0 0.0 0.0"/>
+            <parent link="inter_1"/>
+            <child link="grip_body"/>
+        </joint>
+    </xacro:macro>
+    <xacro:combined_model/>
 </robot>
