Commit message: made changes in urdf file

File: gripper_pkg/urdf/grip.urdf (robot description, URDF)
Before this commit: robot grip, 4 links, 3 joints
Joints:
- joint slide_left: origin xyz=0 0 0 rpy=0 0 0  -> xyz=-0.025 0 0.24 rpy=0 0 0 
- joint slide_right: origin xyz=0 0 0 rpy=0 0 0  -> xyz=0.025 0 0.24 rpy=0 0 0 
